Commit message: improve urdf

File: src/arm.urdf (robot description, URDF)
Before this commit: robot omnipointer, 9 links, 8 joints
Joints:
- joint arm_joint_3: origin xyz=0 0 0.187 rpy=0 1.57 0 -> xyz=0.02 0 0.187 rpy=0 1.57 0

Commit message: first prototype

File: src/arm.urdf (robot description, URDF)
Before this commit: robot omnipointer, 9 links, 8 joints
Links:
- link tip: geometry collision sphere radius=0.01; visual sphere radius=0.04
Joints:
- joint arm_joint_7: origin xyz=0 0 0.115 rpy=0 0 0 -> xyz=0 0 0.04 rpy=3.14 0 0

Commit message: version tested on tiago

File: src/arm.urdf (robot description, URDF)
Before this commit: robot omnipointer, 9 links, 8 joints
Joints:
- joint arm_joint_0: origin xyz=0 0 0 rpy=0 0 0 -> xyz=0 0 0 rpy=0 0 3.1415
- joint arm_joint_7: origin xyz=0 0 0.04 rpy=3.14 0 0 -> xyz=0 0 0.04 rpy=3.1415 0. 0.

Commit message: Update URDF with new dimensions, some elements still need adjustment
- Modified URDF file to reflect the new dimensions of the arm components
- Updated joint positions and link lengths according to the latest design
- Some elements still require further adjustments for final accuracy

File: src/arm.urdf (robot description, URDF)
Before this commit: robot omnipointer, 9 links, 8 joints
Links:
- link arm_link_2: geometry collision box size=0.0356 0.05 0.2050; visual box size=0.0356 0.05 0.2050
- link arm_link_3: geometry collision box size=0.0356 0.05 0.160; visual box size=0.0356 0.05 0.160
Joints:
- joint arm_joint_3: origin xyz=0.02 0 0.187 rpy=0 1.57 0 -> xyz=0.02 0 0.2050 rpy=0 1.57 0

Commit message: Correct movement for the arms and urdf model

File: src/arm.urdf (robot description, URDF)
Before this commit: robot omnipointer, 9 links, 8 joints
Links:
- link arm_link_1: geometry collision box size=0.0402 0.05 0.123; visual box size=0.0402 0.05 0.111
- link arm_link_3: geometry collision box size=0.0356 0.05 0.200; visual box size=0.0356 0.05 0.200
- link arm_link_4: geometry collision box size=0.0356 0.05 0.08; visual box size=0.0356 0.05 0.03
Joints:
- joint arm_joint_3: origin xyz=0.02 0 0.2050 rpy=0 1.57 0 -> xyz=0.0250 0 0.2050 rpy=0 1.57 0
- joint arm_joint_4: origin xyz=0 0 0.165 rpy=0 0 0.0 -> xyz=0 0 0.200 rpy=0 0 0.0
- joint arm_joint_5: origin xyz=0 0 0.08 rpy=0 1.57 0 -> xyz=0 0 0.04 rpy=0 1.57 0

Commit message: Update URDF and add arguments for each side of the arm
- Updated URDF file to support the new configuration
- Added arguments to handle left and right sides of the arm independently
- Ensured compatibility with the teleoperation setup for dual-arm control

File: src/arm.urdf (robot description, URDF)
Before this commit: robot omnipointer, 9 links, 8 joints
Links:
- link arm_link_0: geometry collision box size=0.1143 0.1143 0.0600; visual box size=0.1143 0.1143 0.0600
- link arm_link_1: geometry collision box size=0.0402 0.05 0.115; visual box size=0.0402 0.05 0.115
- link arm_link_2: geometry collision box size=0.0356 0.05 0.2060; visual box size=0.0356 0.05 0.2060
- link arm_link_3: geometry collision box size=0.0356 0.05 0.200; visual box size=0.0356 0.05 0.198
- link arm_link_4: geometry collision box size=0.0356 0.05 0.03; visual box size=0.0356 0.05 0.03
Joints:
- joint arm_joint_1: origin xyz=0 0 0.0545 rpy=0 0 0.0 -> xyz=0 0 0.0600 rpy=0 0 0.0
- joint arm_joint_2: origin xyz=0 0 0.123 rpy=0 0.0 0 -> xyz=0 0 0.115 rpy=0 0.0 0
- joint arm_joint_5: origin xyz=0 0 0.04 rpy=0 1.57 0 -> xyz=0 0 0.045 rpy=0 1.57 0

Commit message: Modify code to publish joint states and handle arm position translation
- Implemented joint state publisher to broadcast current joint positions
- Added functionality to translate the initial position of the arm and the current position
- Ensured proper synchronization between initial and actual positions for accurate teleoperation
- Improved feedback for better control and monitoring of the robot arm

File: src/arm.urdf (robot description, URDF)
Before this commit: robot omnipointer, 9 links, 8 joints
Links:
- link arm_link_2: geometry collision box size=0.0356 0.05 0.2050; visual box size=0.0356 0.05 0.2050
- link arm_link_3: geometry collision box size=0.0356 0.05 0.1975; visual box size=0.0356 0.05 0.1975
- link arm_link_5: geometry collision box size=0.0356 0.05 0.045; visual box size=0.0356 0.05 0.0425
- link arm_link_6: geometry collision box size=0.0356 0.05 0.093; visual box size=0.0356 0.05 0.093
Joints:
- joint arm_joint_0: origin xyz=0 0 0 rpy=0 0 3.1415 -> xyz=0 0 0 rpy=0 0 0
- joint arm_joint_3: origin xyz=0.0250 0 0.2050 rpy=0 1.57 0 -> xyz=0.026 0 0.2050 rpy=0 1.57 0
- joint arm_joint_4: origin xyz=0 0 0.200 rpy=0 0 0.0 -> xyz=0 0 0.1975 rpy=0 0 0.0
- joint arm_joint_5: origin xyz=0 0 0.045 rpy=0 1.57 0 -> xyz=0 0 0.0425 rpy=0 1.57 0
- joint arm_joint_7: origin xyz=0 0 0.04 rpy=3.1415 0. 0. -> xyz=0 0 0.093 rpy=3.1415 0. 3.1415
